File: PCB/CDS.kicad_sch (KiCad schematic)
At the start: 38 parts, among them Q1 2N7002, SW1 Magic Switch, U1 STM32F401CBUx, U2 XC6206PxxxMR, Y1 8 MHz

Commit message: Updated sheets
Other:
- company: Cipulot PCB Design  -> LU.SV Solutions
